Commit message: added the the forarm link

File: src/my_robot_description/urdf/arm.xacro (robot description, xacro)
@@ -7,4 +7,6 @@
     <xacro:property name="base_width" value="0.4" />
     <xacro:property name="base_height" value="0.2" />
+    <xacro:property name="arm_radius" value="0.02" />
+    <xacro:property name="arm_length" value="0.3" />
     <link name="arm_base">
         <visual>
@@ -28,4 +30,24 @@
                            o_rpy="0 0 0"/>
     </link>
+    <xacro:macro name="arm" params="prefix">
+        <link name="${prefix}_link">
+            <visual>
+                <geometry>
+                    <cylinder radius="${arm_radius}" length="${arm_length}" />
+                </geometry>
+                <origin xyz="0 0 ${arm_length / 2.0 }" rpy="0 0 0" />
+                <material name="orange" />
+            </visual>
+            <collision>
+                <geometry>
+                    <origin xyz="0 0 ${arm_length / 2.0 }" rpy="0 0 0" />
+                </geometry>
+                <origin xyz="0 0 0" rpy="0 0 0" />
+            </collision>
+            <xacro:cylinder_inertia m="1.0" r="${arm_radius}" l="${arm_length}"
+                           o_xyz="0 0 ${arm_length / 2.0 }" o_rpy="0 0 0"/>
+        </link>
+    </xacro:macro>
+    <xacro:arm prefix="forearm" />
     <joint name="base_arm_base" type="fixed">
         <parent link="base_link" />
@@ -35,3 +57,12 @@
             rpy="0 0 0" />
     </joint>
+    <joint name="arm_base_forearm" type="revolute">
+        <parent link="arm_base" />
+        <child link="forearm_link" />
+        <origin
+            xyz="0 0 ${robot_base_height}"
+            rpy="0 0 0" />
+        <axis xyz="0 1 0"/>
+        <limit lower="-1.57" upper="1.57" effort="5" velocity="1.0"/>
+    </joint>
 </robot>

Commit message: modified arm joints limit

File: src/my_robot_description/urdf/arm.xacro (robot description, xacro)
@@ -50,4 +50,5 @@
     </xacro:macro>
     <xacro:arm prefix="forearm" />
+    <xacro:arm prefix="hand" />
     <joint name="base_arm_base" type="fixed">
         <parent link="base_link" />
@@ -64,5 +65,16 @@
             rpy="0 0 0" />
         <axis xyz="0 1 0"/>
-        <limit lower="-1.57" upper="1.57" effort="5" velocity="1.0"/>
+        <limit lower="0" upper="1.57" effort="100" velocity="100"/>
+        <dynamics friction="0.3" damping="0.3" />
+    </joint>
+    <joint name="forearm_hand" type="revolute">
+        <parent link="forearm_link" />
+        <child link="hand_link" />
+        <origin
+            xyz="0 0 ${arm_length}"
+            rpy="0 0 0" />
+        <axis xyz="0 1 0"/>
+        <limit lower="0" upper="1.57" effort="100" velocity="100"/>
+        <dynamics friction="0.3" damping="0.3" />
     </joint>
 </robot>
